File: schematic/amc.sch (KiCad schematic (older format))
At the start: 2 parts

Commit message: Schema di base
Parts:
- removed U?: P8, MODULE, symbol P8
- added D?: RG16080B-BIY-V, MODULE, symbol RG16080B-BIY-V
- added J?: MCP23017, MODULE, symbol MCP23017
Connections:
- wire segments 0 -> 23
Changed lines of the file:
@@
 LIBS:memory
 LIBS:xilinx
-LIBS:special
 LIBS:microcontrollers
 LIBS:dsp
@@
 LIBS:valves
 LIBS:MyBeagleBone
-EELAYER 27 0
+LIBS:amc-cache
+EELAYER 25 0
 EELAYER END
 $Descr A4 11693 8268
@@
 $EndDescr
 $Comp
-L P8 U?
-U 1 1 553E7EEB
-P 6000 3750
-F 0 "U?" H 6000 3650 50  0000 C CNN
-F 1 "P8" H 6000 3850 50  0000 C CNN
-F 2 "MODULE" H 6000 3750 50  0001 C CNN
-F 3 "DOCUMENTATION" H 6000 3750 50  0001 C CNN
-	1    6000 3750
+L P9 U?
+U 1 1 553E7EFA
+P 2950 5600
+F 0 "U?" H 2950 5500 50  0000 C CNN
+F 1 "P9" H 2950 5700 50  0000 C CNN
+F 2 "MODULE" H 2950 5600 50  0001 C CNN
+F 3 "DOCUMENTATION" H 2950 5600 50  0001 C CNN
+	1    2950 5600
 	1    0    0    -1
 $EndComp
 $Comp
-L P9 U?
-U 1 1 553E7EFA
-P 3900 3750
-F 0 "U?" H 3900 3650 50  0000 C CNN
-F 1 "P9" H 3900 3850 50  0000 C CNN
-F 2 "MODULE" H 3900 3750 50  0001 C CNN
-F 3 "DOCUMENTATION" H 3900 3750 50  0001 C CNN
-	1    3900 3750
+L MCP23017 J?
+U 1 1 5549E7C6
+P 5000 5150
+F 0 "J?" H 5000 5050 50  0000 C CNN
+F 1 "MCP23017" H 5000 5250 50  0000 C CNN
+F 2 "MODULE" H 5000 5150 50  0001 C CNN
+F 3 "DOCUMENTATION" H 5000 5150 50  0001 C CNN
+	1    5000 5150
 	1    0    0    -1
 $EndComp
+$Comp
+L RG16080B-BIY-V D?
+U 1 1 554B4170
+P 7150 3250
+F 0 "D?" H 7150 3400 50  0000 C CNN
+F 1 "RG16080B-BIY-V" H 7150 3500 50  0000 C CNN
+F 2 "MODULE" H 7150 3250 50  0001 C CNN
+F 3 "DOCUMENTATION" H 7150 3250 50  0001 C CNN
+	1    7150 3250
+	1    0    0    -1
+$EndComp
+Wire Wire Line
+	4250 5700 3700 5700
+Wire Wire Line
+	3700 5600 4250 5600
+Wire Wire Line
+	4250 5400 4100 5400
+Wire Wire Line
+	4100 5400 4100 4500
+Wire Wire Line
+	4100 4500 3700 4500
+Wire Wire Line
+	5750 4500 7500 4500
+Wire Wire Line
+	7500 4500 7500 3700
+Wire Wire Line
+	7400 3700 7400 4600
+Wire Wire Line
+	7400 4600 5750 4600
+Wire Wire Line
+	5750 4700 7300 4700
+Wire Wire Line
+	7300 4700 7300 3700
+Wire Wire Line
+	5750 4800 7200 4800
+Wire Wire Line
+	7200 4800 7200 3700
+Wire Wire Line
+	5750 4900 7100 4900
+Wire Wire Line
+	7100 4900 7100 3700
+Wire Wire Line
+	7000 3700 7000 5000
+Wire Wire Line
+	7000 5000 5750 5000
+Wire Wire Line
+	6900 3700 6900 5100
+Wire Wire Line
+	6900 5100 5750 5100
+Wire Wire Line
+	5750 5200 6800 5200
+Wire Wire Line
+	6800 5200 6800 3700
+Wire Wire Line
+	6200 3700 3700 3700
+Wire Wire Line
+	3700 3700 3700 4500
 $EndSCHEMATC

Commit message: Collegato alla 5V
Connections:
- wire segments 23 -> 29
Changed lines of the file:
@@
 Wire Wire Line
 	3700 3700 3700 4500
+Wire Wire Line
+	3700 4800 3950 4800
+Wire Wire Line
+	3950 4800 3950 5300
+Wire Wire Line
+	3950 5300 4250 5300
+Wire Wire Line
+	6300 3700 6300 3900
+Wire Wire Line
+	6300 3900 3800 3900
+Wire Wire Line
+	3800 3900 3800 4800
+Connection ~ 3800 4800
 $EndSCHEMATC

Commit message: Schematico Logico
Parts:
- removed D?: RG16080B-BIY-V, MODULE, symbol RG16080B-BIY-V
- removed J?: MCP23017, MODULE, symbol MCP23017
- removed U?: P9, MODULE, symbol P9
- added C?: 1uF, symbol C
- added D?: RG16080B-BIY-V_LOGIC, MODULE, symbol RG16080B-BIY-V_LOGIC
- added D? (x16): LED, symbol LED
- added J?: MCP23017_LOGIC, MODULE, symbol MCP23017_LOGIC
- added R? (x16): 220, symbol R
- added RV?: 20K, symbol POT
- added U? (x2): 74HC595, symbol 74HC595
- added U?: P9_I2C_SPI, symbol P9_I2C_SPI
Connections:
- net labels added: +5V, GND, VCC
- wire segments 29 -> 97
