File: eagle_file/MODULO2_1.sch (EAGLE design)
At the start: 59 parts, among them IC1 74HC595N

Commit message: Fix Modulo 0
Pin all'esterno della scheda
Parts:
- removed JP2: (no value), SparkFun-Connectors:M01PTH
- added JP11: (no value), SparkFun-Connectors:M06LOCK
Connections:
- removed net N$33: IC1A.QH*, JP2.1
- new net QH: IC1A.QH*, JP11.4
- net CS: now also JP11.2
- net GND: now also JP11.1
- net SCLK: now also JP11.5
- net SDI: now also JP11.3
- net VCC: now also JP11.6
Changed lines of the file:
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@@
 <part name="SUPPLY9" library="SparkFun-Aesthetics" deviceset="VCC" device=""/>
 <part name="GND9" library="SparkFun-Aesthetics" deviceset="GND" device=""/>
-<part name="JP2" library="SparkFun-Connectors" deviceset="M01" device="PTH"/>
 <part name="T9" library="transistor" deviceset="*-NPN-" device="TO92-EBC"/>
 <part name="R1" library="resistor" deviceset="R-EU_" device="R0805"/>
@@
 <part name="JP9" library="SparkFun-Connectors" deviceset="M02" device="2.54MM_SCREWTERM"/>
 <part name="JP10" library="SparkFun-Connectors" deviceset="M02" device="2.54MM_SCREWTERM"/>
+<part name="JP11" library="SparkFun-Connectors" deviceset="M06" device="LOCK"/>
+<part name="SUPPLY10" library="SparkFun-Aesthetics" deviceset="VCC" device=""/>
+<part name="GND10" library="SparkFun-Aesthetics" deviceset="GND" device=""/>
 </parts>
 <sheets>
@@
 <instance part="SUPPLY9" gate="G$1" x="5.08" y="116.84"/>
 <instance part="GND9" gate="1" x="5.08" y="88.9"/>
-<instance part="JP2" gate="G$1" x="73.66" y="76.2" rot="R90"/>
 <instance part="T9" gate="G$1" x="93.98" y="60.96" rot="R270"/>
 <instance part="R1" gate="G$1" x="93.98" y="132.08" rot="R90"/>
@@
 <instance part="JP9" gate="G$1" x="175.26" y="27.94" rot="R90"/>
 <instance part="JP10" gate="G$1" x="119.38" y="27.94" rot="R90"/>
+<instance part="JP11" gate="G$1" x="58.42" y="58.42" rot="MR0"/>
+<instance part="SUPPLY10" gate="G$1" x="40.64" y="71.12"/>
+<instance part="GND10" gate="1" x="40.64" y="48.26"/>
 </instances>
 <busses>
@@
 <junction x="116.84" y="144.78"/>
 </segment>
+<segment>
+<pinref part="SUPPLY10" gate="G$1" pin="VCC"/>
+<wire x1="40.64" y1="71.12" x2="40.64" y2="66.04" width="0.1524" layer="91"/>
+<pinref part="JP11" gate="G$1" pin="6"/>
+<wire x1="40.64" y1="66.04" x2="53.34" y2="66.04" width="0.1524" layer="91"/>
+</segment>
 </net>
 <net name="GND" class="0">
@@
 <pinref part="GND2" gate="1" pin="GND"/>
 <wire x1="154.94" y1="144.78" x2="160.02" y2="144.78" width="0.1524" layer="91"/>
+</segment>
+<segment>
+<pinref part="GND10" gate="1" pin="GND"/>
+<wire x1="40.64" y1="50.8" x2="40.64" y2="53.34" width="0.1524" layer="91"/>
+<pinref part="JP11" gate="G$1" pin="1"/>
+<wire x1="40.64" y1="53.34" x2="53.34" y2="53.34" width="0.1524" layer="91"/>
 </segment>
 </net>
@@
 <label x="35.56" y="106.68" size="1.778" layer="95"/>
 </segment>
+<segment>
+<pinref part="JP11" gate="G$1" pin="5"/>
+<wire x1="53.34" y1="63.5" x2="40.64" y2="63.5" width="0.1524" layer="91"/>
+<label x="45.72" y="63.5" size="1.778" layer="95"/>
+</segment>
 </net>
 <net name="SDO" class="0">
@@
 <label x="2.54" y="104.14" size="1.778" layer="95"/>
 </segment>
+<segment>
+<pinref part="JP11" gate="G$1" pin="3"/>
+<wire x1="53.34" y1="58.42" x2="40.64" y2="58.42" width="0.1524" layer="91"/>
+<label x="45.72" y="58.42" size="1.778" layer="95"/>
+</segment>
 </net>
 <net name="CS" class="0">
@@
 <label x="35.56" y="99.06" size="1.778" layer="95"/>
 </segment>
-</net>
-<net name="N$33" class="0">
+<segment>
+<pinref part="JP11" gate="G$1" pin="2"/>
+<wire x1="53.34" y1="55.88" x2="40.64" y2="55.88" width="0.1524" layer="91"/>
+<label x="45.72" y="55.88" size="1.778" layer="95"/>
+</segment>
+</net>
+<net name="QH" class="0">
 <segment>
 <pinref part="IC1" gate="A" pin="QH*"/>
-<pinref part="JP2" gate="G$1" pin="1"/>
 <wire x1="68.58" y1="88.9" x2="73.66" y2="88.9" width="0.1524" layer="91"/>
-<wire x1="73.66" y1="88.9" x2="73.66" y2="83.82" width="0.1524" layer="91"/>
-</segment>
-</net>
+<label x="68.58" y="88.9" size="1.778" layer="95"/>
+</segment>
+<segment>
+<pinref part="JP11" gate="G$1" pin="4"/>
+<wire x1="53.34" y1="60.96" x2="40.64" y2="60.96" width="0.1524" layer="91"/>
+<label x="45.72" y="60.96" size="1.778" layer="95"/>
+</segment>
+</net>
