File: eagle_file/MODULO2_def.brd (EAGLE design)
At the start: 160 x 100 mm, 59 parts, among them IC1 74HC595N

Commit message: MODULO2_def
Parts:
- added R17, R18: (no value), SparkFun-Resistors:0805
Connections:
- new net OUTPUT: JP11.4, R17.1
- net QH: now also R17.2, R18.2; no longer JP11.4
- net SDI: now also R18.1
Routing:
- net VCC: track 0.00 -> 660.7 mm
- net SCLK: track 0.00 -> 163.4 mm
- net SDI: track 0.00 -> 146.7 mm
- net N$46: track 0.00 -> 109.5 mm
- net GND: track 0.00 -> 108.8 mm, vias 0 -> 20
- net N$40: track 0.00 -> 107.4 mm
- net CS: track 0.00 -> 98.4 mm
- net N$30: track 0.00 -> 91.7 mm
- net N$38: track 0.00 -> 78.3 mm
- net N$39: track 0.00 -> 78.2 mm
- net N$26: track 0.00 -> 71.8 mm
- net N$3: track 0.00 -> 71.2 mm
- net N$1: track 0.00 -> 69.9 mm
- net N$55: track 0.00 -> 65.9 mm
- net N$34: track 0.00 -> 65.0 mm
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