File: eagle_file/MODULO2_def.brd (EAGLE design)
At the start: 160 x 100 mm, 61 parts, among them IC1 74HC595N

Commit message: Fix PDF
Ho tolto alcuni layer inutili dal pdf dei PCB
Parts:
- moved D1 7.62 mm to (134.6, 50.8)
- moved D10 7.62 mm to (62.2, 78.7)
- moved D11 7.62 mm to (45.7, 50.8)
- moved D12 7.62 mm to (44.5, 78.7)
- moved D13 7.62 mm to (27.9, 50.8)
- moved D14 7.62 mm to (26.7, 78.7)
- moved D15 7.62 mm to (10.2, 50.8)
- moved D16 7.62 mm to (8.89, 78.7)
- moved D2 7.62 mm to (133.3, 78.7)
- moved D3 7.62 mm to (116.8, 50.8)
- moved D4 7.62 mm to (115.6, 78.7)
- moved D5 7.62 mm to (99.1, 50.8)
- moved D6 7.62 mm to (97.8, 78.7)
- moved D7 7.62 mm to (81.3, 50.8)
- moved D8 7.62 mm to (80.0, 78.7)
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Other:
- board size 160 x 100 mm -> 147.3 x 92.4 mm
