File: eagle_file/MODULO2_def.sch (EAGLE design)
At the start: 61 parts, among them IC1 74HC595N

Commit message: MODULO2_def
Parts:
- R17, R18: device SparkFun-Passives:RESISTOR0805-RES -> SparkFun-Resistors:RESISTOR0805-RES
Connections:
- new net OUTPUT: JP11.4, R17.1
- net QH: no longer JP11.4
- net SDI: now also R18.1
Other:
- moved on the sheet: R17, R18
