File: eagle_file/MODULO1.brd (EAGLE design)
At the start: 55.9 x 69.5 mm, 6 parts, among them IC1 MCP23017SP

Commit message: Modulo1
Routing:
- net N$13: track 105.9 -> 20.9 mm
- net N$12: track 97.9 -> 174.6 mm
- net N$11: track 90.1 -> 21.3 mm
- net N$10: track 82.4 -> 20.9 mm
- net N$9: track 74.7 -> 21.3 mm
- net N$8: track 66.6 -> 21.7 mm
- net N$4: track 12.2 -> 51.3 mm
- net N$3: track 20.2 -> 57.3 mm
- net N$5: track 12.2 -> 46.9 mm
- net N$7: track 58.6 -> 24.6 mm
- net N$6: track 48.2 -> 27.9 mm
- net N$17: track 27.4 -> 9.72 mm
- net N$2: track 20.8 -> 29.7 mm
- net N$21: track 77.9 -> 69.1 mm
- net N$14: track 115.9 -> 107.8 mm
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Other:
- board text added: "BOTTOM"
