File: eagle_file/MODULO1.sch (EAGLE design)
At the start: 6 parts, among them IC1 MCP23017SP

Commit message: Modulo 0 pdf
Modulo 0 senza contorno ai fori
Connections:
- net GND: now also U$2.GND@7
Changed lines of the file:
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@@
 <wire x1="116.84" y1="81.28" x2="116.84" y2="73.66" width="0.1524" layer="91"/>
+</segment>
+<segment>
+<pinref part="U$2" gate="G$1" pin="GND@7"/>
+<pinref part="GND2" gate="1" pin="GND"/>
+<wire x1="-22.86" y1="48.26" x2="-20.32" y2="48.26" width="0.1524" layer="91"/>
+<wire x1="-20.32" y1="48.26" x2="-20.32" y2="45.72" width="0.1524" layer="91"/>
 </segment>
 </net>
