File: eagle_file/MODULO2_pp.brd (EAGLE design)
At the start: 71.1 x 94.9 mm, 34 parts, among them IC1 74HC595N

Commit message: Modulo2
Parts:
- JP1, JP11, JP6: device SparkFun-Connectors:1X06_LOCK -> SparkFun-Connectors:1X06
Routing:
- net VCC: track 349.4 -> 424.0 mm
- net N$41: track 92.8 -> 33.7 mm
- net GND: track 43.3 -> 87.3 mm, vias 6 -> 12
- net N$11: track 35.6 -> 6.67 mm
- net SCLK: track 82.9 -> 56.0 mm
- net N$13: track 30.6 -> 55.7 mm
- net N$4: track 28.9 -> 5.40 mm
- net SDI: track 63.8 -> 85.3 mm
- net N$6: track 56.1 -> 38.6 mm
- net N$7: track 51.7 -> 38.6 mm
- net N$33: track 34.3 -> 45.0 mm
- net N$38: track 35.0 -> 45.1 mm
- net CS: track 100.3 -> 92.3 mm
- net N$43: track 29.4 -> 21.6 mm
- net N$10: track 45.7 -> 38.6 mm
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Other:
- board text added: "BTM"
