File: eagle_file/MODULO2_ps.brd (EAGLE design)
At the start: 73.6 x 67 mm, 29 parts

Commit message: Modulo2
Parts:
- JP1: device SparkFun-Connectors:1X06_LOCK -> SparkFun-Connectors:1X06
Routing:
- net VCC: track 355.7 -> 282.4 mm
- net N$49: track 94.0 -> 26.4 mm
- net N$54: track 83.8 -> 36.8 mm
- net N$20: track 39.8 -> 76.0 mm
- net N$23: track 105.1 -> 74.6 mm
- net N$45: track 61.0 -> 34.9 mm
- net N$27: track 6.87 -> 30.8 mm
- net N$24: track 6.86 -> 29.9 mm
- net N$21: track 6.75 -> 28.0 mm
- net GND: track 59.5 -> 41.2 mm
- net N$26: track 55.4 -> 72.6 mm
- net N$17: track 68.9 -> 77.8 mm
- net N$46: track 23.1 -> 27.1 mm
- net N$47: track 33.1 -> 35.8 mm
- net N$51: track 37.3 -> 34.8 mm
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