File: eagle_file/MODULO2_ps.sch (EAGLE design)
At the start: 29 parts

Commit message: Modulo2
Parts:
- JP1: device SparkFun-Connectors:M06LOCK -> SparkFun-Connectors:M06SILK_FEMALE_PTH
Changed lines of the file:
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@@
 <part name="JP9" library="SparkFun-Connectors" deviceset="M03" device="-SCREW-5MM"/>
 <part name="GND1" library="SparkFun-Aesthetics" deviceset="GND" device=""/>
-<part name="JP1" library="SparkFun-Connectors" deviceset="M06" device="LOCK"/>
+<part name="JP1" library="SparkFun-Connectors" deviceset="M06" device="SILK_FEMALE_PTH"/>
 <part name="SUPPLY1" library="SparkFun-Aesthetics" deviceset="VCC" device=""/>
 </parts>
